File: 2024/倒立振子/KiCad _Data/Main/Main.kicad_sch (KiCad schematic)
At the start: 17 parts, among them J1 Conn_01x03_Socket, J2 Conn_01x04_Socket, J3 Conn_01x04_Socket, SW1 SW_Push, SW2 SW_Push

Commit message: 基板データの更新
Parts:
- removed D1, D2: D, symbol Device:D
- removed SW2: SW_Push, symbol Switch:SW_Push
- added SW1: SW_Push, Button_Switch_THT:SW_PUSH_6mm, symbol Switch:SW_Push
- C1, C2: footprint (none) -> Capacitor_THT:CP_Radial_D5.0mm_P2.50mm
- J1: renamed from J2; footprint (none) -> Connector_JST:JST_XH_B4B-XH-A_1x04_P2.50mm_Vertical
- J2: renamed from J3; footprint (none) -> Connector_JST:JST_XH_B4B-XH-A_1x04_P2.50mm_Vertical
- J3: renamed from J1; footprint (none) -> Connector_JST:JST_XH_B3B-XH-A_1x03_P2.50mm_Vertical
- R1: renamed from R3; footprint (none) -> Resistor_THT:R_Axial_DIN0204_L3.6mm_D1.6mm_P5.08mm_Horizontal
- R2: renamed from R1; footprint (none) -> Resistor_THT:R_Axial_DIN0204_L3.6mm_D1.6mm_P5.08mm_Horizontal
- R3: renamed from R2; footprint (none) -> Resistor_THT:R_Axial_DIN0204_L3.6mm_D1.6mm_P5.08mm_Horizontal
- SW2: renamed from SW1; footprint (none) -> Button_Switch_THT:SW_PUSH_6mm
- U1: renamed from U4; footprint (none) -> Connector_PinHeader_2.54mm:PinHeader_1x07_P2.54mm_Horizontal
- U2: renamed from U3; footprint (none) -> L3GD20H_Module:L3GD20H_Module
- U3: renamed from U1; footprint (none) -> A4988:A4988
- U4: renamed from U2; footprint (none) -> A4988:A4988
Connections:
- net +12V: now also J3.1 (Pin_1)
- net +5V: now also J3.3 (Pin_3), SW1.1
- net M1_DIR: now also A1.7 (D4); no longer A1.6 (D3)
- net M1_STEP: now also A1.6 (D3); no longer A1.5 (D2)
- net M2_DIR: now also A1.9 (D6); no longer A1.8 (D5)
- net M2_STEP: now also A1.8 (D5); no longer A1.7 (D4)
- net at A1.10 (D7): now also SW1.2
- no-connect marks 26 -> 19
