File: 2024/倒立振子/KiCad _Data/PSU/PSU/PSU.kicad_pcb (KiCad board)
At the start: 2 copper layers, 64 x 68 mm, 14 parts, among them J1 Conn_01x03_Socket, SW1 SW_DIP_x01, U1 AMS1117-5.0

Commit message: 基板データの更新
Parts:
- MES1: moved to B.Cu
- moved C1 0.51 mm to (154.5, 107.2)
- moved C4 0.51 mm to (162.7, 107.2)
- turned MES1 to 180 degrees
Routing:
- net GND: track 0.00 -> 195.8 mm
- net Net-(D1-K): track 0.00 -> 46.6 mm
- net +12V: track 0.00 -> 43.7 mm
- net +5V: track 0.00 -> 28.9 mm
- net Net-(BT1-+): track 0.00 -> 9.89 mm
- net Net-(D4-K): track 0.00 -> 4.68 mm
- net Net-(D3-K): track 0.00 -> 4.43 mm
Other:
- outline, holes or cut-outs redrawn
