File: 2024/自立無線/ハードウェア/KiCadData/Kicker_Board/Kicker_Board.kicad_pcb (KiCad board)
At the start: 2 copper layers, 56.9 x 61.5 mm, 11 parts, among them J1 Conn_01x02_Socket, J2 Conn_01x02_Socket, J3 Conn_01x02_Socket, J4 Conn_01x02_Socket, Q1 NMOS, U1 XL6009

Commit message: 色々
ああああああああああああ
Parts:
- removed J2, J3: Conn_01x02_Socket, Connector_JST:JST_XH_B2B-XH-A_1x02_P2.50mm_Vertical
- added REF**: PinHeader_1x01_P1.00mm_Vertical, Connector_PinHeader_1.00mm:PinHeader_1x01_P1.00mm_Vertical, F.Cu at (160.0, 107.2)
- added REF**: PinHeader_1x01_P1.00mm_Vertical, Connector_PinHeader_1.00mm:PinHeader_1x01_P1.00mm_Vertical, F.Cu at (152.4, 114.8)
- added REF**: PinHeader_1x01_P1.00mm_Vertical, Connector_PinHeader_1.00mm:PinHeader_1x01_P1.00mm_Vertical, F.Cu at (161.8, 105.5)
- added REF**: PinHeader_1x01_P1.00mm_Vertical, Connector_PinHeader_1.00mm:PinHeader_1x01_P1.00mm_Vertical, F.Cu at (154.3, 113.2)
- J1, J4: footprint Connector_JST:JST_XH_B2B-XH-A_1x02_P2.50mm_Vertical -> Connector_PinHeader_2.54mm:PinHeader_1x02_P2.54mm_Vertical
- moved Q1 38.3 mm to (154.4, 104.1), turned to -90 degrees
- moved R2 27.0 mm to (122.0, 106.7), turned to 0 degrees
- moved R1 26.6 mm to (122.0, 104.1), turned to 0 degrees
- turned J1 to 0 degrees
- turned J4 to 0 degrees
Routing:
- net Net-(D1-K): track 0.00 -> 247.1 mm
- net GND: track 0.00 -> 170.8 mm
- net Net-(D2-A): track 0.00 -> 139.4 mm
- net Net-(J3-Pin_1): track 0.00 -> 116.2 mm
- net /FET1: track 0.00 -> 43.4 mm
- net Net-(D2-K): track 0.00 -> 32.4 mm
- net +12V: track 0.00 -> 27.0 mm
- net Net-(Q1-G): track 0.00 -> 13.6 mm
